File: controller/controller/controller.kicad_pcb (KiCad board)
At the start: 2 copper layers, 132.3 x 120.4 mm, 52 parts, among them J1-I1 SJ-3524-SMT, J11-O1 SJ-3524-SMT, SW1 SW_Omron_B3FS, U1 H11L1, U2 74HC4051, U3 Pico, U4 I2S_PCM_51XX_SOUNDCARD

Commit message: update to v2
Parts:
- DISP1, SW1, TP1, TP10, TP11, TP12, TP2, TP3, TP4, TP5, TP6, TP7, TP8, TP9: moved to F.Cu
- RV1, RV2, RV3, RV4, RV5, RV6, RV7, RV8: footprint Potentiometer_THT:Potentiometer_Alps_RK09K_Single_Vertical -> MIDI_projects:Potentiometer_Alps_RK09K_Single_Vertical; moved to F.Cu
- moved U3 107.4 mm to (79.8, 47.2)
- moved R13 91.1 mm to (72.1, 77.3), turned to -90 degrees
- moved R17 90.9 mm to (83.0, 77.3), turned to -90 degrees
- moved R7 90.4 mm to (108.3, 47.0), turned to -90 degrees
- moved R8 90.3 mm to (105.8, 47.0), turned to -90 degrees
- moved TP1 89.2 mm to (77.5, 101.1), turned to 0 degrees
- moved TP5 87.3 mm to (77.5, 116.2), turned to 0 degrees
- moved TP9 86.7 mm to (77.4, 131.5), turned to 0 degrees
- moved RV7 85.0 mm to (79.6, 80.7)
- moved RV2 83.9 mm to (150.1, 61.8)
- moved R9 83.4 mm to (77.5, 77.3), turned to -90 degrees
- moved R20 79.7 mm to (154.0, 77.3), turned to -90 degrees
- moved U4 77.7 mm to (156.6, 40.3), turned to 90 degrees
- moved SW1 70.0 mm to (144.2, 50.2), turned to 90 degrees
- moved RV3 69.9 mm to (103.8, 61.9)
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Connections:
- net Net-(U2-A) renamed /AIN
- U2 pad 13: /POT3 -> /POT2
- U2 pad 5: /POT2 -> /POT3
- U3 pad 10: /TPAD3 -> /TPAD11
- U3 pad 11: /TPAD2 -> /TPAD3
- U3 pad 12: /TPAD1 -> /TPAD7
- U3 pad 14: /TPAD8 -> /TPAD10
- U3 pad 15: /TPAD7 -> /TPAD2
- U3 pad 17: /TPAD5 -> /TPAD9
- U3 pad 19: /TPAD9 -> /TPAD1
- U3 pad 20: /TPAD10 -> /TPAD5
- U3 pad 21: /TPAD11 -> /TPAD4
- U3 pad 27: /I2S_LRCK -> /I2S_BCK
- U3 pad 9: /TPAD4 -> /TPAD8
Routing:
- net GND: track 427.0 -> 40.8 mm, vias 6 -> 4
- net +3V3: track 545.4 -> 303.4 mm, vias 2 -> 1
- net /SDA: track 158.4 -> 24.8 mm
- net /SCL: track 154.2 -> 27.9 mm, vias 1 -> 0
- net /POT3: track 119.2 -> 12.0 mm
- net /TPAD12: track 213.6 -> 131.3 mm, vias 1 -> 2
- net /AS0: track 66.8 -> 0.00 mm, vias 2 -> 0
- net /POT2: track 97.9 -> 34.0 mm
- net /AS1: track 63.2 -> 0.00 mm, vias 2 -> 0
- net /AS2: track 59.1 -> 0.00 mm, vias 2 -> 0
- net /POT1: track 66.6 -> 9.97 mm
- net unconnected-(D1-K-Pad1): track 7.39 -> 57.9 mm, vias 0 -> 2
- net /MIDI input 1/RX: track 67.2 -> 116.5 mm
- net Net-(D1-A): track 24.0 -> 71.0 mm
- net /AIN: track 82.1 -> 36.2 mm, vias 2 -> 1
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- added copper zone on B.Cu, net GND
- removed copper zone on F.Cu, net GND
Other:
- board size 132.3 x 120.4 mm -> 97.3 x 120.4 mm
