File: controller/controller/_autosave-controller.kicad_sch (KiCad schematic)
At the start: 40 parts, among them SW1 SW_Omron_B3FS, U2 74HC4051, U3 Pico, U4 I2S_PCM_51XX_SOUNDCARD

Commit message: prototype 1 sent to production
Parts:
- C1: LCSC (none) -> C14663
- DISP1, U3, U4: now not fitted; now left out of the parts list
- R10, R11, R12, R13, R14, R15, R16, R17, R18, R19, R20, R9: LCSC (none) -> C17514
- R7, R8: LCSC (none) -> C17673
- RV1, RV2, RV3, RV4, RV5, RV6, RV7, RV8: LCSC (none) -> C209770
- SW1: LCSC (none) -> C2888769
- TP1, TP10, TP11, TP12, TP2, TP3, TP4, TP5, TP6, TP7, TP8, TP9: now not fitted
- U2: LCSC (none) -> C9386
Connections:
- net GND: now also U3.28 (GND), U3.38 (GND)
- net I2S_BCK: no longer U3.26 (GPIO20)
- net I2S_LRCK: now also U3.26 (GPIO20)
