File: controller/controller/controller.kicad_sch (KiCad schematic)
At the start: 40 parts, among them SW1 SW_Omron_B3FS, U2 74HC4051, U3 Pico, U4 I2S_PCM_51XX_SOUNDCARD

Commit message: update to v2
Parts:
- U3: footprint RPi_Pico:RPi_Pico_SMD_TH -> MIDI_projects:RPi_Pico_SMD_TH
Connections:
- net I2S_BCK: now also U3.27 (GPIO21)
- net I2S_LRCK: no longer U3.27 (GPIO21)
- net POT2: now also U2.13 (A0); no longer U2.5 (A5)
- net POT3: now also U2.5 (A5); no longer U2.13 (A0)
- net TPAD1: now also U3.19 (GPIO14); no longer U3.12 (GPIO9)
- net TPAD10: now also U3.14 (GPIO10); no longer U3.20 (GPIO15)
- net TPAD11: now also U3.10 (GPIO7); no longer U3.21 (GPIO16)
- net TPAD2: now also U3.15 (GPIO11); no longer U3.11 (GPIO8)
- net TPAD3: now also U3.11 (GPIO8); no longer U3.10 (GPIO7)
- net TPAD4: now also U3.21 (GPIO16); no longer U3.9 (GPIO6)
- net TPAD5: now also U3.20 (GPIO15); no longer U3.17 (GPIO13)
- net TPAD7: now also U3.12 (GPIO9); no longer U3.15 (GPIO11)
- net TPAD8: now also U3.9 (GPIO6); no longer U3.14 (GPIO10)
- net TPAD9: now also U3.17 (GPIO13); no longer U3.19 (GPIO14)
- net AIN: now reaches U2.3 (A), U3.34 (GPIO28_ADC2)
Other:
- company: (none) -> bjonnh.net
- title: (none) -> EMMG Midi controller
Changed lines of the file:
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@@
 	(generator_version "8.0")
 	(paper "A4")
+	(title_block
+		(title "EMMG Midi controller")
+		(rev "1")
+		(company "bjonnh.net")
+	)
 	(wire
 		(pts
@@
 		)
 	)
-	(label "TPAD8"
+	(label "TPAD10"
 		(at 167.64 100.33 0)
 		(fields_autoplaced yes)
@@
 		)
 	)
-	(label "TPAD10"
+	(label "TPAD5"
 		(at 167.64 115.57 0)
 		(fields_autoplaced yes)
@@
 		)
 	)
-	(label "POT3"
+	(label "POT2"
 		(at 252.73 82.55 0)
 		(fields_autoplaced yes)
@@
 		)
 	)
-	(label "TPAD9"
+	(label "TPAD1"
 		(at 167.64 113.03 0)
 		(fields_autoplaced yes)
@@
 		)
 	)
-	(label "TPAD3"
+	(label "TPAD11"
 		(at 167.64 90.17 0)
 		(fields_autoplaced yes)
@@
 		)
 	)
-	(label "TPAD11"
+	(label "TPAD4"
 		(at 212.09 115.57 0)
 		(fields_autoplaced yes)
@@
 		)
 	)
-	(label "TPAD5"
+	(label "TPAD9"
 		(at 167.64 107.95 0)
 		(fields_autoplaced yes)
@@
 		)
 	)
-	(label "TPAD7"
+	(label "TPAD2"
 		(at 167.64 102.87 0)
 		(fields_autoplaced yes)
@@
 		)
 	)
-	(label "POT2"
+	(label "POT3"
 		(at 252.73 95.25 0)
 		(fields_autoplaced yes)
@@
 		)
 	)
-	(label "TPAD2"
+	(label "TPAD3"
 		(at 167.64 92.71 0)
 		(fields_autoplaced yes)
@@
 		)
 	)
-	(label "TPAD1"
+	(label "AIN"
+		(at 222.25 82.55 0)
+		(fields_autoplaced yes)
+		(effects
+			(font
+				(size 1.27 1.27)
+			)
+			(justify left bottom)
+		)
+	)
+	(label "TPAD7"
 		(at 167.64 95.25 0)
 		(fields_autoplaced yes)
@@
 		)
 	)
-	(label "TPAD4"
+	(label "TPAD8"
 		(at 167.64 87.63 0)
 		(fields_autoplaced yes)
@@
 		)
 	)
-	(label "I2S_LRCK"
+	(label "I2S_BCK"
 		(at 210.82 100.33 0)
 		(fields_autoplaced yes)
@@
 			)
 		)
-		(property "Footprint" "RPi_Pico:RPi_Pico_SMD_TH"
+		(property "Footprint" "MIDI_projects:RPi_Pico_SMD_TH"
 			(at 191.77 91.44 90)
 			(effects

Commit message: prototype 1 sent to production
Parts:
- DISP1, U3, U4: now not fitted; now left out of the parts list
- RV1, RV2, RV3, RV4, RV5, RV6, RV7, RV8: footprint Potentiometer_THT:Potentiometer_Alps_RK09K_Single_Vertical -> MIDI_projects:Potentiometer_Alps_RK09K_Single_Vertical
Connections:
- net GND: now also U3.28 (GND), U3.38 (GND)
- net I2S_BCK: no longer U3.26 (GPIO20)
- net I2S_LRCK: now also U3.26 (GPIO20)
Changed lines of the file:
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@@
 	(wire
 		(pts
+			(xy 209.55 72.39) (xy 219.71 72.39)
+		)
+		(stroke
+			(width 0)
+			(type default)
+		)
+	)
+	(wire
+		(pts
 			(xy 248.92 87.63) (xy 252.73 87.63)
 		)
@@
 	(wire
 		(pts
+			(xy 209.55 97.79) (xy 223.52 97.79)
+		)
+		(stroke
+			(width 0)
+			(type default)
+		)
+	)
+	(wire
+		(pts
 			(xy 22.86 54.61) (xy 30.48 54.61)
 		)
@@
 		)
 	)
-	(label "I2S_BCK"
+	(label "I2S_LRCK"
 		(at 210.82 102.87 0)
 		(fields_autoplaced yes)
@@
 			)
 		)
-		(property "Footprint" "Potentiometer_THT:Potentiometer_Alps_RK09K_Single_Vertical"
+		(property "Footprint" "MIDI_projects:Potentiometer_Alps_RK09K_Single_Vertical"
 			(at 34.29 97.79 0)
 			(effects
@@
 			)
 		)
-		(property "Footprint" "Potentiometer_THT:Potentiometer_Alps_RK09K_Single_Vertical"
+		(property "Footprint" "MIDI_projects:Potentiometer_Alps_RK09K_Single_Vertical"
 			(at 34.29 119.38 0)
 			(effects
@@
 	)
 	(symbol
-		(lib_id "MIDI_projects:Pico")
-		(at 191.77 91.44 0)
+		(lib_id "power:GND")
+		(at 219.71 72.39 0)
 		(unit 1)
 		(exclude_from_sim no)
@@
 		(dnp no)
 		(fields_autoplaced yes)
+		(property "Reference" "#PWR049"
+			(at 219.71 78.74 0)
+			(effects
+				(font
+					(size 1.27 1.27)
+				)
+				(hide yes)
+			)
+		)
+		(property "Value" "GND"
+			(at 219.71 77.47 0)
+			(effects
+				(font
+					(size 1.27 1.27)
+				)
+			)
+		)
+		(property "Footprint" ""
+			(at 219.71 72.39 0)
+			(effects
+				(font
+					(size 1.27 1.27)
+				)
+				(hide yes)
+			)
+		)
+		(property "Datasheet" ""
+			(at 219.71 72.39 0)
+			(effects
+				(font
+					(size 1.27 1.27)
+				)
+				(hide yes)
+			)
+		)
+		(property "Description" "Power symbol creates a global label with name \"GND\" , ground"
+			(at 219.71 72.39 0)
+			(effects
+				(font
+					(size 1.27 1.27)
+				)
+				(hide yes)
+			)
+		)
+		(pin "1"
+		)
+		(instances
+			(project "controller"
+				(path "/3acbb1c1-c637-462c-af9e-3f63db2c37c2"
+					(reference "#PWR049")
+					(unit 1)
+				)
+			)
+		)
+	)
+	(symbol
+		(lib_id "MIDI_projects:Pico")
+		(at 191.77 91.44 0)
+		(unit 1)
+		(exclude_from_sim no)
+		(in_bom no)
+		(on_board yes)
+		(dnp yes)
+		(fields_autoplaced yes)
 		(property "Reference" "U3"
 			(at 191.77 59.69 0)
@@
 			)
 		)
-		(property "Footprint" "Potentiometer_THT:Potentiometer_Alps_RK09K_Single_Vertical"
+		(property "Footprint" "MIDI_projects:Potentiometer_Alps_RK09K_Single_Vertical"
 			(at 34.29 54.61 0)
 			(effects
@@
 			)
 		)
-		(property "Footprint" "Potentiometer_THT:Potentiometer_Alps_RK09K_Single_Vertical"
+		(property "Footprint" "MIDI_projects:Potentiometer_Alps_RK09K_Single_Vertical"
 			(at 34.29 139.7 0)
 			(effects
@@
 			)
 		)
-		(property "Footprint" "Potentiometer_THT:Potentiometer_Alps_RK09K_Single_Vertical"
+		(property "Footprint" "MIDI_projects:Potentiometer_Alps_RK09K_Single_Vertical"
 			(at 34.29 160.02 0)
 			(effects
@@
 	)
 	(symbol
+		(lib_id "power:GND")
+		(at 223.52 97.79 0)
+		(unit 1)
+		(exclude_from_sim no)
+		(in_bom yes)
+		(on_board yes)
+		(dnp no)
+		(fields_autoplaced yes)
+		(property "Reference" "#PWR048"
+			(at 223.52 104.14 0)
+			(effects
+				(font
+					(size 1.27 1.27)
+				)
+				(hide yes)
+			)
+		)
+		(property "Value" "GND"
+			(at 223.52 102.87 0)
+			(effects
+				(font
+					(size 1.27 1.27)
+				)
+			)
+		)
+		(property "Footprint" ""
+			(at 223.52 97.79 0)
+			(effects
+				(font
+					(size 1.27 1.27)
+				)
+				(hide yes)
+			)
+		)
+		(property "Datasheet" ""
+			(at 223.52 97.79 0)
+			(effects
+				(font
+					(size 1.27 1.27)
+				)
+				(hide yes)
+			)
+		)
+		(property "Description" "Power symbol creates a global label with name \"GND\" , ground"
+			(at 223.52 97.79 0)
+			(effects
+				(font
+					(size 1.27 1.27)
+				)
+				(hide yes)
+			)
+		)
+		(pin "1"
+		)
+		(instances
+			(project "controller"
+				(path "/3acbb1c1-c637-462c-af9e-3f63db2c37c2"
+					(reference "#PWR048")
+					(unit 1)
+				)
+			)
+		)
+	)
+	(symbol
 		(lib_id "Device:R_Potentiometer")
 		(at 34.29 33.02 0)
@@
 			)
 		)
-		(property "Footprint" "Potentiometer_THT:Potentiometer_Alps_RK09K_Single_Vertical"
+		(property "Footprint" "MIDI_projects:Potentiometer_Alps_RK09K_Single_Vertical"
 			(at 34.29 33.02 0)
 			(effects
@@
 		(on_board yes)
 		(dnp no)
-		(fields_autoplaced yes)
 		(property "Reference" "#PWR09"
 			(at 214.63 81.28 0)
@@
 		)
 		(property "Value" "+3V3"
-			(at 214.63 72.39 0)
+			(at 214.122 73.914 0)
 			(effects
 				(font
@@
 			)
 		)
-		(property "Footprint" "Potentiometer_THT:Potentiometer_Alps_RK09K_Single_Vertical"
+		(property "Footprint" "MIDI_projects:Potentiometer_Alps_RK09K_Single_Vertical"
 			(at 34.29 180.34 0)
 			(effects
@@
 		(unit 1)
 		(exclude_from_sim no)
-		(in_bom yes)
+		(in_bom no)
 		(on_board yes)
-		(dnp no)
+		(dnp yes)
 		(property "Reference" "U4"
 			(at 236.22 52.07 0)
@@
 		(unit 1)
 		(exclude_from_sim no)
-		(in_bom yes)
+		(in_bom no)
 		(on_board yes)
-		(dnp no)
+		(dnp yes)
 		(property "Reference" "DISP1"
 			(at 78.74 38.1 0)
@@
 			)
 		)
-		(property "Footprint" "Potentiometer_THT:Potentiometer_Alps_RK09K_Single_Vertical"
+		(property "Footprint" "MIDI_projects:Potentiometer_Alps_RK09K_Single_Vertical"
 			(at 34.29 76.2 0)
 			(effects

Commit message: Mure Stoff
Parts:
- C1: LCSC (none) -> C14663
- R10, R11, R12, R13, R14, R15, R16, R17, R18, R19, R20, R9: LCSC (none) -> C17514
- R7, R8: LCSC (none) -> C17673
- RV1, RV2, RV3, RV4, RV5, RV6, RV7, RV8: LCSC (none) -> C209770
- SW1: LCSC (none) -> C2888769
- TP1, TP10, TP11, TP12, TP2, TP3, TP4, TP5, TP6, TP7, TP8, TP9: now not fitted
- U2: LCSC (none) -> C9386

Commit message: Merged
Parts:
- DISP1, TP1, TP10, TP11, TP12, TP2, TP3, TP4, TP5, TP6, TP7, TP8, TP9, U3, U4: now fitted
Changed lines of the file:
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@@
 		(in_bom yes)
 		(on_board yes)
-		(dnp yes)
+		(dnp no)
 		(property "Reference" "TP4"
 			(at 115.57 137.922 0)
@@
 		(in_bom yes)
 		(on_board yes)
-		(dnp yes)
+		(dnp no)
 		(property "Reference" "TP1"
 			(at 62.23 137.922 0)
@@
 		(in_bom no)
 		(on_board yes)
-		(dnp yes)
+		(dnp no)
 		(fields_autoplaced yes)
 		(property "Reference" "U3"
@@
 		(in_bom yes)
 		(on_board yes)
-		(dnp yes)
+		(dnp no)
 		(property "Reference" "TP5"
 			(at 133.35 137.922 0)
@@
 		(in_bom yes)
 		(on_board yes)
-		(dnp yes)
+		(dnp no)
 		(property "Reference" "TP12"
 			(at 257.81 137.922 0)
@@
 		(in_bom yes)
 		(on_board yes)
-		(dnp yes)
+		(dnp no)
 		(property "Reference" "TP2"
 			(at 80.01 137.922 0)
@@
 		(in_bom yes)
 		(on_board yes)
-		(dnp yes)
+		(dnp no)
 		(property "Reference" "TP6"
 			(at 151.13 137.922 0)
@@
 		(in_bom yes)
 		(on_board yes)
-		(dnp yes)
+		(dnp no)
 		(property "Reference" "TP9"
 			(at 204.47 137.922 0)
@@
 		(in_bom yes)
 		(on_board yes)
-		(dnp yes)
+		(dnp no)
 		(property "Reference" "TP11"
 			(at 240.03 137.922 0)
@@
 		(in_bom yes)
 		(on_board yes)
-		(dnp yes)
+		(dnp no)
 		(property "Reference" "TP7"
 			(at 168.91 137.922 0)
@@
 		(in_bom yes)
 		(on_board yes)
-		(dnp yes)
+		(dnp no)
 		(property "Reference" "TP3"
 			(at 97.79 137.922 0)
@@
 		(in_bom no)
 		(on_board yes)
-		(dnp yes)
+		(dnp no)
 		(property "Reference" "U4"
 			(at 236.22 52.07 0)
@@
 		(in_bom yes)
 		(on_board yes)
-		(dnp yes)
+		(dnp no)
 		(property "Reference" "TP10"
 			(at 222.25 137.922 0)
@@
 		(in_bom no)
 		(on_board yes)
-		(dnp yes)
+		(dnp no)
 		(property "Reference" "DISP1"
 			(at 78.74 38.1 0)
@@
 		(in_bom yes)
 		(on_board yes)
-		(dnp yes)
+		(dnp no)
 		(property "Reference" "TP8"
 			(at 186.69 137.922 0)
