File: controller/controller/midi_output.kicad_sch (KiCad schematic)
At the start: 5 parts, among them J11-O1 SJ-3524-SMT

Commit message: update to v2
Parts:
- J11-O1: footprint SJ-3524-SMT:CUI_SJ-3524-SMT -> MIDI_projects:CUI_SJ-3524-SMT
Changed lines of the file:
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@@
 	(wire
 		(pts
-			(xy 100.33 100.33) (xy 100.33 95.25)
+			(xy 100.33 95.25) (xy 100.33 100.33)
 		)
 		(stroke
@@
 	(wire
 		(pts
+			(xy 110.49 85.09) (xy 144.78 85.09)
+		)
+		(stroke
+			(width 0)
+			(type default)
+		)
+	)
+	(wire
+		(pts
+			(xy 90.17 105.41) (xy 114.3 105.41)
+		)
+		(stroke
+			(width 0)
+			(type default)
+		)
+	)
+	(wire
+		(pts
+			(xy 100.33 100.33) (xy 144.78 100.33)
+		)
+		(stroke
+			(width 0)
+			(type default)
+		)
+	)
+	(wire
+		(pts
+			(xy 90.17 105.41) (xy 90.17 102.87)
+		)
+		(stroke
+			(width 0)
+			(type default)
+		)
+	)
+	(wire
+		(pts
+			(xy 144.78 85.09) (xy 144.78 97.79)
+		)
+		(stroke
+			(width 0)
+			(type default)
+		)
+	)
+	(wire
+		(pts
 			(xy 121.92 105.41) (xy 144.78 105.41)
-		)
-		(stroke
-			(width 0)
-			(type default)
-		)
-	)
-	(wire
-		(pts
-			(xy 110.49 85.09) (xy 144.78 85.09)
-		)
-		(stroke
-			(width 0)
-			(type default)
-		)
-	)
-	(wire
-		(pts
-			(xy 90.17 105.41) (xy 114.3 105.41)
-		)
-		(stroke
-			(width 0)
-			(type default)
-		)
-	)
-	(wire
-		(pts
-			(xy 90.17 105.41) (xy 90.17 102.87)
-		)
-		(stroke
-			(width 0)
-			(type default)
-		)
-	)
-	(wire
-		(pts
-			(xy 100.33 100.33) (xy 144.78 100.33)
-		)
-		(stroke
-			(width 0)
-			(type default)
-		)
-	)
-	(wire
-		(pts
-			(xy 144.78 85.09) (xy 144.78 97.79)
 		)
 		(stroke
@@
 			)
 		)
-		(property "Footprint" "SJ-3524-SMT:CUI_SJ-3524-SMT"
+		(property "Footprint" "MIDI_projects:CUI_SJ-3524-SMT"
 			(at 155.194 92.71 0)
 			(effects
@@
 		(lib_id "power:GND")
 		(at 110.49 85.09 0)
+		(mirror y)
 		(unit 1)
 		(exclude_from_sim no)
@@
 		(on_board yes)
 		(dnp no)
-		(fields_autoplaced yes)
 		(property "Reference" "#PWR010"
 			(at 110.49 91.44 0)

Commit message: prototype 1 sent to production
Parts:
- J11-O1: now not fitted
Other:
- moved on the sheet: DT1
Changed lines of the file:
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@@
+	(wire
+		(pts
+			(xy 90.17 87.63) (xy 100.33 87.63)
+		)
+		(stroke
+			(width 0)
+			(type default)
+		)
+	)
+	(wire
+		(pts
+			(xy 100.33 100.33) (xy 144.78 100.33)
+		)
+		(stroke
+			(width 0)
+			(type default)
+		)
+	)
+	(wire
+		(pts
+			(xy 90.17 105.41) (xy 90.17 104.14)
+		)
+		(stroke
+			(width 0)
+			(type default)
+		)
+	)
+	(wire
+		(pts
+			(xy 144.78 85.09) (xy 144.78 97.79)
+		)
+		(stroke
+			(width 0)
+			(type default)
+		)
+	)
+	(wire
+		(pts
+			(xy 121.92 105.41) (xy 144.78 105.41)
+		)
+		(stroke
+			(width 0)
+			(type default)
+		)
+	)
+	(wire
+		(pts
+			(xy 90.17 95.25) (xy 90.17 96.52)
+		)
+		(stroke
+			(width 0)
+			(type default)
+		)
+	)
 	(wire
 		(pts
 			(xy 90.17 105.41) (xy 114.3 105.41)
-		)
-		(stroke
-			(width 0)
-			(type default)
-		)
-	)
-	(wire
-		(pts
-			(xy 100.33 100.33) (xy 144.78 100.33)
-		)
-		(stroke
-			(width 0)
-			(type default)
-		)
-	)
-	(wire
-		(pts
-			(xy 90.17 105.41) (xy 90.17 102.87)
-		)
-		(stroke
-			(width 0)
-			(type default)
-		)
-	)
-	(wire
-		(pts
-			(xy 144.78 85.09) (xy 144.78 97.79)
-		)
-		(stroke
-			(width 0)
-			(type default)
-		)
-	)
-	(wire
-		(pts
-			(xy 121.92 105.41) (xy 144.78 105.41)
-		)
-		(stroke
-			(width 0)
-			(type default)
-		)
-	)
-	(wire
-		(pts
-			(xy 90.17 87.63) (xy 100.33 87.63)
 		)
 		(stroke
@@
 	(symbol
 		(lib_id "Device:LED")
-		(at 90.17 99.06 90)
+		(at 90.17 100.33 90)
 		(unit 1)
 		(exclude_from_sim no)
@@
 		(dnp no)
 		(property "Reference" "DT1"
-			(at 93.98 99.3774 90)
+			(at 93.98 100.6474 90)
 			(effects
 				(font
@@
 		)
 		(property "Value" "LED"
-			(at 93.98 101.9174 90)
+			(at 93.98 103.1874 90)
 			(effects
 				(font
@@
 		)
 		(property "Footprint" "LED_SMD:LED_0603_1608Metric"
-			(at 87.122 98.552 0)
+			(at 87.122 99.822 0)
 			(effects
 				(font
@@
 		)
 		(property "Datasheet" "~"
-			(at 90.17 99.06 0)
+			(at 90.17 100.33 0)
 			(effects
 				(font
@@
 		)
 		(property "Description" "Light emitting diode"
-			(at 90.17 99.06 0)
+			(at 90.17 100.33 0)
 			(effects
 				(font
@@
 		)
 		(property "LCSC" "C72038"
-			(at 90.17 99.06 90)
+			(at 90.17 100.33 90)
 			(effects
 				(font
@@
 		)
 		(instances
-			(project "minimidi_v1"
-				(path "/7c6c2d1f-d81f-45f2-99e6-075fc53a5e89/e41d1471-dfd4-454e-991d-302e3492a1d2"
+			(project "controller"
+				(path "/3acbb1c1-c637-462c-af9e-3f63db2c37c2/e41d1471-dfd4-454e-991d-302e3492a1d2"
 					(reference "R3")
 					(unit 1)
@@
 		(in_bom no)
 		(on_board yes)
-		(dnp no)
+		(dnp yes)
 		(property "Reference" "J11-O1"
 			(at 157.48 90.17 0)

Commit message: Mure Stoff
Parts:
- R1: LCSC C17634 -> C17634
Changed lines of the file:
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@@
 			)
 		)
-		(property "LCSC" " C17634 "
+		(property "LCSC" "C17634 "
 			(at 100.33 91.44 0)
 			(effects

Commit message: Merged
Parts:
- J11-O1: now fitted
Changed lines of the file:
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@@
 		(in_bom no)
 		(on_board yes)
-		(dnp yes)
+		(dnp no)
 		(property "Reference" "J11-O1"
 			(at 157.48 90.17 0)
